File: CAN Bus Hub 16/CAN Bus Hub.kicad_pcb (KiCad board)
At the start: 2 copper layers, 185 x 15 mm, 24 parts, among them J1 Conn_01x02, J10 Conn_01x02, J11 Conn_01x02, J12 Conn_01x02, J13 Conn_01x02, J14 Conn_01x02, J15 Conn_01x02, J16 Conn_01x02, J2 Conn_01x02, J3 Conn_01x02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

Commit message: Added Board Information
Other:
- board text added: "Can Bus Hub 12 Rev 1 Corwin Hansen"
Changed lines of the file:
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@@
   (general
     (thickness 1.6)
-    (drawings 6)
+    (drawings 7)
     (tracks 87)
     (zones 0)
@@
     (pad 1 np_thru_hole circle (at 0 0) (size 4.3 4.3) (drill 4.3) (layers *.Cu *.Mask))
   )
+  (gr_text "Can Bus Hub 12   Rev 1   Corwin Hansen" (at 105 70) (layer F.SilkS)
+    (effects (font (size 1.5 1.5) (thickness 0.3)))
+  )
   (dimension 15 (width 0.3) (layer Dwgs.User)

Commit message: Reduced solder mask clearance
Other:
- rule pad_to_mask_clearance: 0.2 -> 0
Changed lines of the file:
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@@
     (pad_size 1.524 1.524)
     (pad_drill 0.762)
-    (pad_to_mask_clearance 0.2)
+    (pad_to_mask_clearance 0)
     (aux_axis_origin 0 0)
     (visible_elements FFFFFF7F)
